File: DeviceHardware/OmniPin/OmniPin.kicad_sch (KiCad schematic)
At the start: 52 parts, among them J1 USB_B_Micro, J2 2-1734839-4, J4 Conn_01x02_Pin, Q1 IRLML6402, Q2 IRLML6244, SW1 RST, SW2 BOOT, SW3 POWER, SW4 NEXT, U1 ESP32-C3-MINI-1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

Commit message: hw panelization
Parts:
- SW2: footprint Connector_PinHeader_1.27mm:PinHeader_1x02_P1.27mm_Vertical -> Jumper:SolderJumper-2_P1.3mm_Open_RoundedPad1.0x1.5mm
Changed lines of the file:
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@@
 			)
 		)
-		(property "Footprint" "Connector_PinHeader_1.27mm:PinHeader_1x02_P1.27mm_Vertical"
+		(property "Footprint" "Jumper:SolderJumper-2_P1.3mm_Open_RoundedPad1.0x1.5mm"
 			(at 81.28 82.55 0)
 			(effects

Commit message: update pcb
Parts:
- SW1, SW4: footprint SW_BT:SW_SPST_B3U-1000P -> SW_BT:SW_SPST_B3U-3000P-B
Changed lines of the file:
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@@
 			)
 		)
-		(property "Footprint" "SW_BT:SW_SPST_B3U-1000P"
+		(property "Footprint" "SW_BT:SW_SPST_B3U-3000P-B"
 			(at 93.98 127 0)
 			(effects
@@
 			)
 		)
-		(property "Footprint" "SW_BT:SW_SPST_B3U-1000P"
+		(property "Footprint" "SW_BT:SW_SPST_B3U-3000P-B"
 			(at 19.05 71.12 0)
 			(effects
